Commit message: camera movements in ball collection bot sort node

File: gcr_diff_robot/model/common_properties.xacro (robot description, xacro)
@@ -1,6 +1,6 @@
 <?xml version="1.0"?>
 <robot xmlns:xacro="http://www.ros.org/wiki/xacro">
-    <xacro:property name="effort" value="10.0" />
-    <xacro:property name="velocity" value="5.0" />
+    <xacro:property name="effort" value="1.0" />
+    <xacro:property name="velocity" value="0.5" />
     <!-- =========== Inertia Calculation for Box =========== -->
     <xacro:macro name="box_intertia" params="m l w h xyz rpy">
